Commit message: add sick_tim551 and mapping_config

File: jackal_description/urdf/accessories.urdf.xacro (robot description, xacro)
@@ -13,4 +13,5 @@
   <!-- This optional plate mounts both the upgraded GPS and the Velodyne 3D LIDAR. -->
   <xacro:include filename="$(find jackal_description)/urdf/accessories/bridge_plate.urdf.xacro" />
+<!-- ########################################################################### -->
   <!-- If enabled, generate the LASER payload (by default, a SICK LMS111). -->
   <xacro:include filename="$(find jackal_description)/urdf/accessories/sick_lms1xx_mount.urdf.xacro" />
@@ -25,4 +26,17 @@
     </joint>
   </xacro:if>
+<!-- #################### -->
+  <!-- If enabled, generate the MAPPING configuration. -->
+  <xacro:include filename="$(find sick_tim)/urdf/sick_tim.urdf.xacro" />
+  <xacro:if value="$(optenv MAPPING 0)">
+    <xacro:sick_tim551 name="laser" ros_topic="scan" />
+    <joint name="$(optenv JACKAL_LASER_MOUNT front)_laser_mount_joint" type="fixed">
+      <origin xyz="$(optenv JACKAL_LASER_OFFSET 0 0 0)"
+              rpy="$(optenv JACKAL_LASER_RPY 0 0 0)" />
+      <parent link="$(optenv JACKAL_LASER_MOUNT front)_mount" />
+      <child link="laser_mount_link" />
+    </joint>
+  </xacro:if>
+<!-- ########################################################################### -->
   <!-- If enabled, generate the upgraded Navsat payload (a Novatel Smart6). -->
   <xacro:include filename="$(find jackal_description)/urdf/accessories/novatel_smart6.urdf.xacro" />

Commit message: loading rplidar urdf

File: jackal_description/urdf/accessories.urdf.xacro (robot description, xacro)
@@ -29,4 +29,5 @@
   <!-- If enabled, generate the MAPPING configuration. -->
   <xacro:include filename="$(find sick_tim)/urdf/sick_tim.urdf.xacro" />
+  <xacro:include filename="$(find rplidar_ros)/urdf/rplidar.urdf.xacro" />
   <xacro:if value="$(optenv MAPPING 0)">
     <xacro:sick_tim551 name="laser" ros_topic="scan" />
@@ -36,4 +37,11 @@
       <parent link="$(optenv JACKAL_LASER_MOUNT front)_mount" />
       <child link="laser_mount_link" />
+    </joint>
+    <xacro:rplidar_a2 name="rplidar_laser" ros_topic="rplidar/scan" />
+    <joint name="$jackal_sicktim_joint" type="fixed">
+      <origin xyz="0.2 0 0"
+              rpy="0 1.5708 0" />
+      <parent link="$(optenv JACKAL_LASER_MOUNT front)_mount" />
+      <child link="rplidar_laser_mount_link" />
     </joint>
   </xacro:if>
